File: key_fob/key_fob.sch (KiCad schematic (older format))
At the start: 22 parts

Commit message: Changed external leds back to not using MOSFET
Parts:
- removed Q? (x2): MMBT3904, Package_TO_SOT_SMD:SOT-23, symbol Transistor_BJT:MMBT3904
- R? (x4): value 30 -> 1.2K
- R? (x2): value 15 -> 1.2K
Connections:
- net +3V3: now also R?.1, R?.1
- net +BATT: no longer R?.1, R?.1
- net CONNECTED_LED: now also D?.1 (K)
- net POWER_LED: now also D?.1 (K)
Other:
- moved on the sheet: D?, R?
Changed lines of the file:
@@
 P 4750 3150
 F 0 "R?" H 4820 3196 50  0000 L CNN
-F 1 "30" H 4820 3105 50  0000 L CNN
+F 1 "1.2K" H 4820 3105 50  0000 L CNN
 F 2 "Resistor_SMD:R_0603_1608Metric_Pad1.05x0.95mm_HandSolder" V 4680 3150 50  0001 C CNN
 F 3 "~" H 4750 3150 50  0001 C CNN
@@
 P 4350 3150
 F 0 "R?" H 4420 3196 50  0000 L CNN
-F 1 "30" H 4420 3105 50  0000 L CNN
+F 1 "1.2K" H 4420 3105 50  0000 L CNN
 F 2 "Resistor_SMD:R_0603_1608Metric_Pad1.05x0.95mm_HandSolder" V 4280 3150 50  0001 C CNN
 F 3 "~" H 4350 3150 50  0001 C CNN
@@
 P 3950 3150
 F 0 "R?" H 4020 3196 50  0000 L CNN
-F 1 "30" H 4020 3105 50  0000 L CNN
+F 1 "1.2K" H 4020 3105 50  0000 L CNN
 F 2 "Resistor_SMD:R_0603_1608Metric_Pad1.05x0.95mm_HandSolder" V 3880 3150 50  0001 C CNN
 F 3 "~" H 3950 3150 50  0001 C CNN
@@
 P 3550 3150
 F 0 "R?" H 3620 3196 50  0000 L CNN
-F 1 "30" H 3620 3105 50  0000 L CNN
+F 1 "1.2K" H 3620 3105 50  0000 L CNN
 F 2 "Resistor_SMD:R_0603_1608Metric_Pad1.05x0.95mm_HandSolder" V 3480 3150 50  0001 C CNN
 F 3 "~" H 3550 3150 50  0001 C CNN
@@
 Wire Wire Line
 	3550 3850 3550 3700
-Text GLabel 2650 3950 3    50   Input ~ 0
+Text GLabel 3150 3850 3    50   Input ~ 0
 CONNECTED_LED
 Text GLabel 6350 3600 2    50   Input ~ 0
@@
 L Device:LED D?
 U 1 1 5E4DA2B1
-P 3000 3550
-F 0 "D?" V 3039 3433 50  0000 R CNN
-F 1 "LED" V 2948 3433 50  0000 R CNN
-F 2 "LED_THT:LED_D5.0mm" H 3000 3550 50  0001 C CNN
-F 3 "~" H 3000 3550 50  0001 C CNN
-	1    3000 3550
+P 3150 3550
+F 0 "D?" V 3189 3433 50  0000 R CNN
+F 1 "LED" V 3098 3433 50  0000 R CNN
+F 2 "LED_THT:LED_D5.0mm" H 3150 3550 50  0001 C CNN
+F 3 "~" H 3150 3550 50  0001 C CNN
+	1    3150 3550
 	0    -1   -1   0
 $EndComp
@@
 L Device:R R?
 U 1 1 5E4DA2B7
-P 3000 3150
-F 0 "R?" H 3070 3196 50  0000 L CNN
-F 1 "15" H 3070 3105 50  0000 L CNN
-F 2 "Resistor_SMD:R_0603_1608Metric_Pad1.05x0.95mm_HandSolder" V 2930 3150 50  0001 C CNN
-F 3 "~" H 3000 3150 50  0001 C CNN
-	1    3000 3150
-	1    0    0    -1
-$EndComp
-Wire Wire Line
-	3000 3300 3000 3400
-Wire Wire Line
-	3000 3000 3000 2900
-$Comp
-L power:+BATT #PWR?
-U 1 1 5E4DA2C6
-P 3000 2900
-F 0 "#PWR?" H 3000 2750 50  0001 C CNN
-F 1 "+BATT" H 3015 3073 50  0000 C CNN
-F 2 "" H 3000 2900 50  0001 C CNN
-F 3 "" H 3000 2900 50  0001 C CNN
-	1    3000 2900
-	1    0    0    -1
-$EndComp
-Wire Wire Line
-	2700 3900 2650 3900
-Wire Wire Line
-	2650 3900 2650 3950
-$Comp
-L power:GND #PWR?
-U 1 1 5E4DA2CD
-P 3000 4300
-F 0 "#PWR?" H 3000 4050 50  0001 C CNN
-F 1 "GND" H 3005 4127 50  0000 C CNN
-F 2 "" H 3000 4300 50  0001 C CNN
-F 3 "" H 3000 4300 50  0001 C CNN
-	1    3000 4300
-	1    0    0    -1
-$EndComp
-Wire Wire Line
-	3000 4100 3000 4300
-$Comp
-L Transistor_BJT:MMBT3904 Q?
-U 1 1 5E4DA2C0
-P 2900 3900
-F 0 "Q?" H 3091 3946 50  0000 L CNN
-F 1 "MMBT3904" H 3091 3855 50  0000 L CNN
-F 2 "Package_TO_SOT_SMD:SOT-23" H 3100 3825 50  0001 L CIN
-F 3 "https://www.fairchildsemi.com/datasheets/2N/2N3904.pdf" H 2900 3900 50  0001 L CNN
-	1    2900 3900
-	1    0    0    -1
-$EndComp
+P 3150 3150
+F 0 "R?" H 3220 3196 50  0000 L CNN
+F 1 "1.2K" H 3220 3105 50  0000 L CNN
+F 2 "Resistor_SMD:R_0603_1608Metric_Pad1.05x0.95mm_HandSolder" V 3080 3150 50  0001 C CNN
+F 3 "~" H 3150 3150 50  0001 C CNN
+	1    3150 3150
+	1    0    0    -1
+$EndComp
+Wire Wire Line
+	3150 3300 3150 3400
+Wire Wire Line
+	3150 3000 3150 2900
 Text GLabel 3550 3850 3    50   Input ~ 0
 HEARTBEAT_LED
@@
 L Device:LED D?
 U 1 1 5E4E79F6
-P 2100 3550
-F 0 "D?" V 2139 3433 50  0000 R CNN
-F 1 "LED" V 2048 3433 50  0000 R CNN
-F 2 "LED_THT:LED_D5.0mm" H 2100 3550 50  0001 C CNN
-F 3 "~" H 2100 3550 50  0001 C CNN
-	1    2100 3550
+P 2750 3550
+F 0 "D?" V 2789 3433 50  0000 R CNN
+F 1 "LED" V 2698 3433 50  0000 R CNN
+F 2 "LED_THT:LED_D5.0mm" H 2750 3550 50  0001 C CNN
+F 3 "~" H 2750 3550 50  0001 C CNN
+	1    2750 3550
 	0    -1   -1   0
 $EndComp
@@
 L Device:R R?
 U 1 1 5E4E79FC
-P 2100 3150
-F 0 "R?" H 2170 3196 50  0000 L CNN
-F 1 "15" H 2170 3105 50  0000 L CNN
-F 2 "Resistor_SMD:R_0603_1608Metric_Pad1.05x0.95mm_HandSolder" V 2030 3150 50  0001 C CNN
-F 3 "~" H 2100 3150 50  0001 C CNN
-	1    2100 3150
-	1    0    0    -1
-$EndComp
-Wire Wire Line
-	2100 3300 2100 3400
-Wire Wire Line
-	2100 3000 2100 2900
-$Comp
-L power:+BATT #PWR?
-U 1 1 5E4E7A04
-P 2100 2900
-F 0 "#PWR?" H 2100 2750 50  0001 C CNN
-F 1 "+BATT" H 2115 3073 50  0000 C CNN
-F 2 "" H 2100 2900 50  0001 C CNN
-F 3 "" H 2100 2900 50  0001 C CNN
-	1    2100 2900
-	1    0    0    -1
-$EndComp
-Wire Wire Line
-	1800 3900 1750 3900
-Wire Wire Line
-	1750 3900 1750 3950
-$Comp
-L power:GND #PWR?
-U 1 1 5E4E7A0C
-P 2100 4300
-F 0 "#PWR?" H 2100 4050 50  0001 C CNN
-F 1 "GND" H 2105 4127 50  0000 C CNN
-F 2 "" H 2100 4300 50  0001 C CNN
-F 3 "" H 2100 4300 50  0001 C CNN
-	1    2100 4300
-	1    0    0    -1
-$EndComp
-Wire Wire Line
-	2100 4100 2100 4300
-$Comp
-L Transistor_BJT:MMBT3904 Q?
-U 1 1 5E4E7A13
-P 2000 3900
-F 0 "Q?" H 2191 3946 50  0000 L CNN
-F 1 "MMBT3904" H 2191 3855 50  0000 L CNN
-F 2 "Package_TO_SOT_SMD:SOT-23" H 2200 3825 50  0001 L CIN
-F 3 "https://www.fairchildsemi.com/datasheets/2N/2N3904.pdf" H 2000 3900 50  0001 L CNN
-	1    2000 3900
-	1    0    0    -1
-$EndComp
-Text GLabel 1750 3950 3    50   Input ~ 0
+P 2750 3150
+F 0 "R?" H 2820 3196 50  0000 L CNN
+F 1 "1.2K" H 2820 3105 50  0000 L CNN
+F 2 "Resistor_SMD:R_0603_1608Metric_Pad1.05x0.95mm_HandSolder" V 2680 3150 50  0001 C CNN
+F 3 "~" H 2750 3150 50  0001 C CNN
+	1    2750 3150
+	1    0    0    -1
+$EndComp
+Wire Wire Line
+	2750 3300 2750 3400
+Wire Wire Line
+	2750 3000 2750 2900
+Text GLabel 2750 3850 3    50   Input ~ 0
 POWER_LED
 $Comp
@@
 Wire Wire Line
 	4150 2900 4350 2900
+$Comp
+L power:+3.3V #PWR?
+U 1 1 5E557B5D
+P 3150 2900
+F 0 "#PWR?" H 3150 2750 50  0001 C CNN
+F 1 "+3.3V" H 3165 3073 50  0000 C CNN
+F 2 "" H 3150 2900 50  0001 C CNN
+F 3 "" H 3150 2900 50  0001 C CNN
+	1    3150 2900
+	1    0    0    -1
+$EndComp
+$Comp
+L power:+3.3V #PWR?
+U 1 1 5E559043
+P 2750 2900
+F 0 "#PWR?" H 2750 2750 50  0001 C CNN
+F 1 "+3.3V" H 2765 3073 50  0000 C CNN
+F 2 "" H 2750 2900 50  0001 C CNN
+F 3 "" H 2750 2900 50  0001 C CNN
+	1    2750 2900
+	1    0    0    -1
+$EndComp
+Wire Wire Line
+	2750 3700 2750 3850
+Wire Wire Line
+	3150 3700 3150 3850
 $EndSCHEMATC

Commit message: Filled out title block and printed rev1 pdf
Other:
- note added: "1"
- note added: "2/25/2020"
- note added: "Key Fob Circuit Design"
Changed lines of the file:
@@
 Wire Wire Line
 	3150 3700 3150 3850
+Text Notes 7350 7500 0    50   ~ 0
+Key Fob Circuit Design
+Text Notes 10600 7650 0    50   ~ 0
+1
+Text Notes 8150 7650 0    50   ~ 0
+2/25/2020
 $EndSCHEMATC

Commit message: Imported schematic into pcb layout
Parts:
- gave numbers to parts that had none: 20
Connections:
- no-connect marks 0 -> 19

Commit message: Got some stuff started for key fod pcb
Connections:
- net +3V3: now also S1.1; no longer S1.2
- net +BATT: now also S1.2; no longer S1.1
- net LED_SW: now also S1.6; no longer S1.5
- net POWER_SW: now also S1.5; no longer S1.6
Changed lines of the file:
@@
 	7600 3550 7900 3550
-$Comp
-L power:+BATT #PWR0101
-U 1 1 5E36659B
-P 8250 2200
-F 0 "#PWR0101" H 8250 2050 50  0001 C CNN
-F 1 "+BATT" H 8265 2373 50  0000 C CNN
-F 2 "" H 8250 2200 50  0001 C CNN
-F 3 "" H 8250 2200 50  0001 C CNN
-	1    8250 2200
-	1    0    0    -1
-$EndComp
 $Comp
 L power:GND #PWR0102
@@
 F 3 "" H 7900 4100 50  0001 C CNN
 	1    7900 4100
-	1    0    0    -1
-$EndComp
-$Comp
-L power:+3.3V #PWR0103
-U 1 1 5E319CC0
-P 8000 2300
-F 0 "#PWR0103" H 8000 2150 50  0001 C CNN
-F 1 "+3.3V" H 8015 2473 50  0000 C CNN
-F 2 "" H 8000 2300 50  0001 C CNN
-F 3 "" H 8000 2300 50  0001 C CNN
-	1    8000 2300
 	1    0    0    -1
 $EndComp
@@
 Text GLabel 2750 3850 3    50   Input ~ 0
 POWER_LED
+Text GLabel 9050 2200 2    50   Input ~ 0
+LED_SW
 Text GLabel 9050 2300 2    50   Input ~ 0
-LED_SW
-Text GLabel 9050 2200 2    50   Input ~ 0
 POWER_SW
 Text GLabel 9050 2400 2    50   Input ~ 0
 SPEAKER_SW
-Wire Wire Line
-	8250 2300 8000 2300
 Text GLabel 4150 2850 1    50   Input ~ 0
 LED_SW
@@
 	1    0    0    -1
 $EndComp
+Wire Wire Line
+	8250 2300 8000 2300
+$Comp
+L power:+3.3V #PWR0103
+U 1 1 5E319CC0
+P 8250 2200
+F 0 "#PWR0103" H 8250 2050 50  0001 C CNN
+F 1 "+3.3V" H 8265 2373 50  0000 C CNN
+F 2 "" H 8250 2200 50  0001 C CNN
+F 3 "" H 8250 2200 50  0001 C CNN
+	1    8250 2200
+	1    0    0    -1
+$EndComp
+$Comp
+L power:+BATT #PWR?
+U 1 1 5E5C3234
+P 8000 2300
+F 0 "#PWR?" H 8000 2150 50  0001 C CNN
+F 1 "+BATT" H 8015 2473 50  0000 C CNN
+F 2 "" H 8000 2300 50  0001 C CNN
+F 3 "" H 8000 2300 50  0001 C CNN
+	1    8000 2300
+	1    0    0    -1
+$EndComp
